File: Paranoid70_PCB/Paranoid70_PCB.kicad_sch (KiCad schematic)
At the start: 72 parts

Commit message: Schema Finish and first go at the PCB
Parts:
- removed D?: D_Small_Filled, symbol Device:D_Small_Filled
- removed MX?: MX-NoLED, symbol MX_alps_hybrid:MX-NoLED
- added D35: D_Small_Filled, Keebio-parts:Diode-hybrid-3pad, symbol Device:D_Small_Filled
- added R1, R2: 4.7kOhm, Keebio-parts:Resistor-Hybrid, symbol Device:R
- added RSW1: RESET SWITCH, Keebio-parts:SW_Tactile_SPST_Angled_MJTP1117, symbol Switch:SW_MEC_5G
- added SW1: RotaryEncoder_Switch, Keebio-parts:RotaryEncoder_EC11, symbol Device:RotaryEncoder_Switch
- D1, D10, D11, D12, D13, D14, D15, D16, D17, D18, D19, D2, D20, D21, D22, D23, D24, D25, D26, D27, D28, D29, D3, D30, D31, D33, D34, D36, D4, D5, D6, D7, D8, D9: renamed from D?; footprint (none) -> Keebio-parts:Diode-hybrid-3pad
- MX1, MX10, MX11, MX12, MX13, MX14, MX15, MX16, MX17, MX18, MX19, MX2, MX20, MX21, MX22, MX23, MX24, MX25, MX26, MX27, MX28, MX29, MX3, MX30, MX31, MX34, MX35, MX4, MX5, MX6, MX7, MX8, MX9: renamed from MX?; footprint (none) -> Keebio-parts:MX-Alps-Choc-1U-NoLED
- MX33: renamed from MX?; footprint (none) -> Keebio-parts:MX-Alps-Choc-2U
- U1: renamed from U?; footprint (none) -> Keebio-parts:Elite-C-castellated-29pin-holes
- U2: renamed from U?; footprint (none) -> Keebio-parts:TRRS-PJ-320A
Connections:
- net +5V: now also U2.3 (RING1), R1.1, R2.1
- net COL7: now also SW1.S2
- net GND: now also U2.2 (TIP), SW1.C
- net ROW5: now also D35.1 (K)
- net at U1.22 (RST): now also RSW1.3 (B), RSW1.4 (B)
- net at U1.23 (GND): now also RSW1.1 (A), RSW1.2 (A)
- net ROT2: now reaches U1.28 (F1)
- net ROT2: now also SW1.B
- net ROT1: now reaches U1.29 (F0)
- net ROT1: now also SW1.A
- net at U1.5 (2/PD1): now also U2.1 (SLEEVE), R2.2
- net at U1.6 (3/PD0): now also U2.4 (RING2), R1.2
- new net: D35.2 (A), SW1.S1
- no-connect marks 0 -> 4
Other:
- added sheet Per Key LED (Per Key LED.kicad_sch)
- moved on the sheet: U2
